Commit message: Add files via upload

File: leo_description/urdf/leo.gazebo.xacro (robot description, xacro)
@@ -116,3 +116,35 @@
     </gazebo>
   </xacro:unless>
+ <!-- LiDAR -->
+  <gazebo reference="base_scan">
+    <sensor type="ray" name="lds_lfcd_sensor">
+      <pose>0 0 0.00 0 0 0</pose>
+      <visualize>true</visualize>
+      <update_rate>5</update_rate>
+      <ray>
+        <scan>
+          <horizontal>
+            <samples>720</samples>
+            <resolution>1</resolution>
+            <min_angle>-1.0472</min_angle>
+            <max_angle>1.0472</max_angle>
+          </horizontal>
+        </scan>
+        <range>
+          <min>0.2</min>
+          <max>5</max>
+          <resolution>0.015</resolution>
+        </range>
+        <noise>
+          <type>gaussian</type>
+          <mean>0.0</mean>
+          <stddev>0.01</stddev>
+        </noise>
+      </ray>
+      <plugin name="gazebo_ros_lds_lfcd_controller" filename="libgazebo_ros_laser.so">
+        <topicName>scan</topicName>
+        <frameName>base_scan</frameName>
+      </plugin>
+    </sensor>
+  </gazebo>
 </robot>

File: leo_description/urdf/leo.urdf.xacro (robot description, xacro)
@@ -120,4 +120,25 @@
   <link name="camera_optical_frame"/>
   <link name="imu_link"/>
+  <link name="base_scan">
+    <visual>
+      <origin xyz="0.04 0 0.0" rpy="1.5707 0 0"/>
+      <geometry>
+        <mesh filename="package://leo_description/models/rplidar.dae" scale="0.001 0.001 0.001" />
+      </geometry>
+    </visual>
+    <collision>
+      <origin xyz=" 0 0 0.0" rpy="1.5707 0 0"/>
+      <geometry>
+        <cylinder length="0.01" radius="0.055"/>
+      </geometry>
+    </collision>
+    <inertial>
+      <mass value="0.114" />
+      <origin xyz="0 0 0" />
+      <inertia ixx="0.001" ixy="0.0" ixz="0.0"
+               iyy="0.001" iyz="0.0"
+               izz="0.001" />
+    </inertial>
+  </link>
   <!-- JOINTS -->
   <joint name="footprint_joint" type="fixed">
@@ -202,4 +223,10 @@
     <child link="imu_link"/>
     <origin xyz="0 0 0" rpy="0 0 0"/>
+  </joint>
+  <!--Scanner Link-->
+  <joint name="scan_joint" type="fixed">
+    <parent link="base_link"/>
+    <child link="base_scan"/>
+    <origin xyz="0.04 0 0.0" rpy="0 0 0"/>
   </joint>
   <!-- TRANSMISSIONS -->
