Commit message: Add files via upload

File: leo_description/urdf/leo.urdf.xacro (robot description, xacro)
@@ -143,5 +143,5 @@
   <!-- JOINTS -->
   <joint name="footprint_joint" type="fixed">
-    <origin xyz="0 0 -0.19783" rpy="0 0 0"/>
+    <origin xyz="0 0 0.15256" rpy="0 0 0"/>
     <child link="base_link"/>
     <parent link="base_footprint"/>

Commit message: Add files via upload

File: leo_description/urdf/leo.urdf.xacro (robot description, xacro)
@@ -143,5 +143,5 @@
   <!-- JOINTS -->
   <joint name="footprint_joint" type="fixed">
-    <origin xyz="0 0 0.15256" rpy="0 0 0"/>
+    <origin xyz="0 0 ${0.15256+0.0625}" rpy="0 0 0"/>
     <child link="base_link"/>
     <parent link="base_footprint"/>
